Commit message: update

File: src/final_project_urdf/urdf/gazebo/my_camera.xacro (robot description, xacro)
@@ -1,9 +1,6 @@
 <robot name="my_sensors" xmlns:xacro="http://wiki.ros.org/xacro">
-  <!-- 被引用的link -->
   <gazebo reference="camera">
-    <!-- 类型设置为 camara -->
     <sensor type="camera" name="camera_node">
-      <update_rate>30.0</update_rate> <!-- 更新频率 -->
-      <!-- 摄像头基本信息设置 -->
+      <update_rate>30.0</update_rate>
       <camera name="head">
         <horizontal_fov>1.3962634</horizontal_fov>

File: src/final_project_urdf/urdf/gazebo/my_move.xacro (robot description, xacro)
@@ -1,4 +1,3 @@
 <robot name="my_car_move" xmlns:xacro="http://wiki.ros.org/xacro">
-    <!-- 传动实现:用于连接控制器与关节 -->
     <xacro:macro name="joint_trans" params="joint_name">
         <!-- Transmission is important to link the joints and the controller -->
@@ -14,8 +13,6 @@
         </transmission>
     </xacro:macro>
-    <!-- 每一个驱动轮都需要配置传动装置 -->
     <xacro:joint_trans joint_name="left_wheel2base_link" />
     <xacro:joint_trans joint_name="right_wheel2base_link" />
-    <!-- 控制器 -->
     <gazebo>
         <plugin name="differential_drive_controller" filename="libgazebo_ros_diff_drive.so">
@@ -28,15 +25,15 @@
             <updateRate>100.0</updateRate>
             <legacyMode>true</legacyMode>
-            <leftJoint>left_wheel2base_link</leftJoint> <!-- 左轮 -->
-            <rightJoint>right_wheel2base_link</rightJoint> <!-- 右轮 -->
-            <wheelSeparation>${base_link_radius * 2}</wheelSeparation> <!-- 车轮间距 -->
-            <wheelDiameter>${wheel_radius * 2}</wheelDiameter> <!-- 车轮直径 -->
+            <leftJoint>left_wheel2base_link</leftJoint>
+            <rightJoint>right_wheel2base_link</rightJoint>
+            <wheelSeparation>${base_link_radius * 2}</wheelSeparation>
+            <wheelDiameter>${wheel_radius * 2}</wheelDiameter>
             <broadcastTF>1</broadcastTF>
             <wheelTorque>30</wheelTorque>
             <wheelAcceleration>1.8</wheelAcceleration>
-            <commandTopic>cmd_vel</commandTopic> <!-- 运动控制话题 -->
+            <commandTopic>cmd_vel</commandTopic>
             <odometryFrame>odom</odometryFrame>
-            <odometryTopic>odom</odometryTopic> <!-- 里程计话题 -->
-            <robotBaseFrame>base_footprint</robotBaseFrame> <!-- 根坐标系 -->
+            <odometryTopic>odom</odometryTopic>
+            <robotBaseFrame>base_footprint</robotBaseFrame>
         </plugin>
     </gazebo>

File: src/final_project_urdf/urdf/my_base.xacro (robot description, xacro)
@@ -1,25 +1,12 @@
-<!--
-    使用 xacro 优化 URDF 版的小车底盘实现：
-    实现思路:
-    1.将一些常量、变量封装为 xacro:property
-      比如:PI 值、小车底盘半径、离地间距、车轮半径、宽度 ....
-    2.使用 宏 封装驱动轮以及支撑轮实现，调用相关宏生成驱动轮与支撑轮
--->
-<!-- 根标签，必须声明 xmlns:xacro -->
 <robot name="my_base" xmlns:xacro="http://www.ros.org/wiki/xacro">
-    <!-- 封装变量、常量 -->
-    <!-- PI 值设置精度需要高一些，否则后续车轮翻转量计算时，可能会出现肉眼不能察觉的车轮倾斜，从而导致模型抖动 -->
     <xacro:property name="PI" value="3.1415926"/>
-    <!-- 宏:黑色设置 -->
     <material name="black">
         <color rgba="0.0 0.0 0.0 1.0" />
     </material>
-    <!-- 底盘属性 -->
-    <xacro:property name="base_footprint_radius" value="0.001" /> <!-- base_footprint 半径  -->
-    <xacro:property name="base_link_radius" value="0.1" /> <!-- base_link 半径 -->
-    <xacro:property name="base_link_length" value="0.08" /> <!-- base_link 长 -->
-    <xacro:property name="earth_space" value="0.015" /> <!-- 离地间距 -->
-    <xacro:property name="base_link_m" value="0.5" /> <!-- 质量  -->
-    <!-- 底盘 -->
+    <xacro:property name="base_footprint_radius" value="0.001" />
+    <xacro:property name="base_link_radius" value="0.1" />
+    <xacro:property name="base_link_length" value="0.08" />
+    <xacro:property name="earth_space" value="0.015" />
+    <xacro:property name="base_link_m" value="0.5" />
     <link name="base_footprint">
       <visual>
@@ -55,10 +42,7 @@
         <material>Gazebo/Yellow</material>
     </gazebo>
-    <!-- 驱动轮 -->
-    <!-- 驱动轮属性 -->
-    <xacro:property name="wheel_radius" value="0.0325" /><!-- 半径 -->
-    <xacro:property name="wheel_length" value="0.015" /><!-- 宽度 -->
-    <xacro:property name="wheel_m" value="0.05" /> <!-- 质量  -->
-    <!-- 驱动轮宏实现 -->
+    <xacro:property name="wheel_radius" value="0.0325" />
+    <xacro:property name="wheel_length" value="0.015" />
+    <xacro:property name="wheel_m" value="0.05" />
     <xacro:macro name="add_wheels" params="name flag">
       <link name="${name}_wheel">
@@ -90,9 +74,6 @@
     <xacro:add_wheels name="left" flag="1" />
     <xacro:add_wheels name="right" flag="-1" />
-    <!-- 支撑轮 -->
-    <!-- 支撑轮属性 -->
-    <xacro:property name="support_wheel_radius" value="0.0075" /> <!-- 支撑轮半径 -->
-    <xacro:property name="support_wheel_m" value="0.03" /> <!-- 质量  -->
-    <!-- 支撑轮宏 -->
+    <xacro:property name="support_wheel_radius" value="0.0075" />
+    <xacro:property name="support_wheel_m" value="0.03" />
     <xacro:macro name="add_support_wheel" params="name flag" >
       <link name="${name}_wheel">

File: src/final_project_urdf/urdf/my_camera.xacro (robot description, xacro)
@@ -1,13 +1,10 @@
-<!-- 摄像头相关的 xacro 文件 -->
 <robot name="my_camera" xmlns:xacro="http://wiki.ros.org/xacro">
-    <!-- 摄像头属性 -->
-    <xacro:property name="camera_length" value="0.01" /> <!-- 摄像头长度(x) -->
-    <xacro:property name="camera_width" value="0.025" /> <!-- 摄像头宽度(y) -->
-    <xacro:property name="camera_height" value="0.025" /> <!-- 摄像头高度(z) -->
-    <xacro:property name="camera_x" value="0.08" /> <!-- 摄像头安装的x坐标 -->
-    <xacro:property name="camera_y" value="0.0" /> <!-- 摄像头安装的y坐标 -->
-    <xacro:property name="camera_z" value="${base_link_length / 2 + camera_height / 2}" /> <!-- 摄像头安装的z坐标:底盘高度 / 2 + 摄像头高度 / 2  -->
-    <xacro:property name="camera_m" value="0.01" /> <!-- 摄像头质量 -->
-    <!-- 摄像头关节以及link -->
+    <xacro:property name="camera_length" value="0.01" />
+    <xacro:property name="camera_width" value="0.025" />
+    <xacro:property name="camera_height" value="0.025" />
+    <xacro:property name="camera_x" value="0.08" />
+    <xacro:property name="camera_y" value="0.0" />
+    <xacro:property name="camera_z" value="${base_link_length / 2 + camera_height / 2}" />
+    <xacro:property name="camera_m" value="0.01" />
     <link name="camera">
         <visual>

File: src/final_project_urdf/urdf/my_laser.xacro (robot description, xacro)
@@ -1,13 +1,9 @@
-<!--
-    小车底盘添加雷达
--->
 <robot name="my_laser" xmlns:xacro="http://wiki.ros.org/xacro">
-    <!-- 雷达支架 -->
-    <xacro:property name="support_length" value="0.15" /> <!-- 支架长度 -->
-    <xacro:property name="support_radius" value="0.01" /> <!-- 支架半径 -->
-    <xacro:property name="support_x" value="0.0" /> <!-- 支架安装的x坐标 -->
-    <xacro:property name="support_y" value="0.0" /> <!-- 支架安装的y坐标 -->
-    <xacro:property name="support_z" value="${base_link_length / 2 + support_length / 2}" /> <!-- 支架安装的z坐标:底盘高度 / 2 + 支架高度 / 2  -->
-    <xacro:property name="support_m" value="0.02" /> <!-- 支架质量 -->
+    <xacro:property name="support_length" value="0.15" />
+    <xacro:property name="support_radius" value="0.01" />
+    <xacro:property name="support_x" value="0.0" />
+    <xacro:property name="support_y" value="0.0" />
+    <xacro:property name="support_z" value="${base_link_length / 2 + support_length / 2}" />
+    <xacro:property name="support_m" value="0.02" />
     <link name="support">
         <visual>
@@ -36,12 +32,10 @@
         <material>Gazebo/White</material>
     </gazebo>
-    <!-- 雷达属性 -->
-    <xacro:property name="laser_length" value="0.05" /> <!-- 雷达长度 -->
-    <xacro:property name="laser_radius" value="0.03" /> <!-- 雷达半径 -->
-    <xacro:property name="laser_x" value="0.0" /> <!-- 雷达安装的x坐标 -->
-    <xacro:property name="laser_y" value="0.0" /> <!-- 雷达安装的y坐标 -->
-    <xacro:property name="laser_z" value="${support_length / 2 + laser_length / 2}" /> <!-- 雷达安装的z坐标:支架高度 / 2 + 雷达高度 / 2  -->
-    <xacro:property name="laser_m" value="0.1" /> <!-- 雷达质量 -->
-    <!-- 雷达关节以及link -->
+    <xacro:property name="laser_length" value="0.05" />
+    <xacro:property name="laser_radius" value="0.03" />
+    <xacro:property name="laser_x" value="0.0" />
+    <xacro:property name="laser_y" value="0.0" />
+    <xacro:property name="laser_z" value="${support_length / 2 + laser_length / 2}" />
+    <xacro:property name="laser_m" value="0.1" />
     <link name="laser">
         <visual>
